Commit message: Tried to add traj controller, not working great.

File: src/ugv_sim/urdf/ugv.urdf.xacro (robot description, xacro)
@@ -71,4 +71,22 @@
     </inertial>
   </link>
+<!-- Dummy Wheel  -->
+<link name="dummy_wheel">
+  <visual>
+    <geometry>
+      <cylinder length="0.02" radius="0.03"/>
+    </geometry>
+    <material name="black"/>
+  </visual>
+  <collision>
+    <geometry>
+      <cylinder length="0.1" radius="0.05"/>
+    </geometry>
+  </collision>
+  <inertial>
+    <mass value="1.0"/>
+    <inertia ixx="0.01" ixy="0.0" ixz="0.0" iyy="0.01" iyz="0.0" izz="0.02"/>
+  </inertial>
+</link>
   <!-- Joints -->
   <!-- Left Wheel Joint -->
@@ -86,4 +104,10 @@
     <axis xyz="0 0 1"/>
   </joint>
+  <!-- Dummy Wheel Joinr  -->
+<joint name="dummy_wheel_joint" type="fixed">
+  <parent link="base_link"/>
+  <child link="dummy_wheel"/>
+  <origin xyz="0.25 0 -0.04" rpy="1.5707 0 -0.02"/>
+</joint>
   <!-- Transmission for wheels -->
   <transmission name="left_wheel_trans">

Commit message: Tried to add traj controller, not working great.

File: src/ugv_sim/urdf/ugv.urdf.xacro (robot description, xacro)
@@ -71,22 +71,4 @@
     </inertial>
   </link>
-<!-- Dummy Wheel  -->
-<link name="dummy_wheel">
-  <visual>
-    <geometry>
-      <cylinder length="0.02" radius="0.03"/>
-    </geometry>
-    <material name="black"/>
-  </visual>
-  <collision>
-    <geometry>
-      <cylinder length="0.1" radius="0.05"/>
-    </geometry>
-  </collision>
-  <inertial>
-    <mass value="1.0"/>
-    <inertia ixx="0.01" ixy="0.0" ixz="0.0" iyy="0.01" iyz="0.0" izz="0.02"/>
-  </inertial>
-</link>
   <!-- Joints -->
   <!-- Left Wheel Joint -->
@@ -104,10 +86,4 @@
     <axis xyz="0 0 1"/>
   </joint>
-  <!-- Dummy Wheel Joinr  -->
-<joint name="dummy_wheel_joint" type="fixed">
-  <parent link="base_link"/>
-  <child link="dummy_wheel"/>
-  <origin xyz="0.25 0 -0.04" rpy="1.5707 0 -0.02"/>
-</joint>
   <!-- Transmission for wheels -->
   <transmission name="left_wheel_trans">

Commit message: Lidar is added.

File: src/ugv_sim/urdf/ugv.urdf.xacro (robot description, xacro)
@@ -71,4 +71,13 @@
     </inertial>
   </link>
+<!-- Lidar Link -->
+<link name="lidar_link">
+  <visual>
+    <geometry>
+      <cylinder length="0.1" radius="${wheel_radius}"/>
+    </geometry>
+    <!-- Add material properties if desired -->
+  </visual>
+</link>
   <!-- Joints -->
   <!-- Left Wheel Joint -->
@@ -85,4 +94,11 @@
     <origin xyz="0 -0.3 -0.02" rpy="1.5707 0 0"/>
     <axis xyz="0 0 1"/>
+  </joint>
+  <!-- Lidar Joint -->
+  <joint name="lidar_joint" type="fixed">
+    <parent link="base_link"/>
+    <child link="lidar_link"/>
+    <!-- Define the origin of the joint -->
+    <origin xyz="0 0 0.1" rpy="0 0 0"/>
   </joint>
   <!-- Transmission for wheels -->
@@ -128,3 +144,29 @@
 </plugin>
   </gazebo>
+<gazebo reference="lidar_link">
+  <sensor type="ray" name="lidar_sensor">
+    <pose>0 0 0 0 0 0</pose>
+    <visualize>true</visualize>
+    <update_rate>10</update_rate>
+    <ray>
+      <scan>
+        <horizontal>
+          <samples>720</samples>
+          <resolution>1</resolution>
+          <min_angle>0</min_angle>
+          <max_angle>1.570796</max_angle>
+        </horizontal>
+      </scan>
+      <range>
+        <min>0.1</min>
+        <max>30.0</max>
+        <resolution>0.01</resolution>
+      </range>
+    </ray>
+    <plugin name="gazebo_ros_laser_controller" filename="libgazebo_ros_laser.so">
+      <topicName>/scan</topicName>
+      <frameName>lidar_link</frameName>
+    </plugin>
+  </sensor>
+</gazebo>
 </robot>

Commit message: Simple fine tunings

File: src/ugv_sim/urdf/ugv.urdf.xacro (robot description, xacro)
@@ -71,4 +71,25 @@
     </inertial>
   </link>
+  <!-- Front Wheel -->
+  <link name="front_wheel">
+  <visual>
+    <geometry>
+      <sphere radius="0.025"/>
+    </geometry>
+    <material name="black"/>
+  </visual>
+  <collision>
+    <geometry>
+      <sphere radius="0.025"/>
+    </geometry>
+  </collision>
+  <inertial>
+    <mass value="1.0"/>
+    <inertia
+      ixx="0.001" ixy="0.0" ixz="0.0"
+      iyy="0.001" iyz="0.0"
+      izz="0.001"/>
+  </inertial>
+</link>
 <!-- Lidar Link -->
 <link name="lidar_link">
@@ -102,4 +123,10 @@
     <origin xyz="0 0 0.1" rpy="0 0 0"/>
   </joint>
+<!-- Front Joint -->
+<joint name="front_wheel_joint" type="fixed">
+  <parent link="base_link"/>
+  <child link="front_wheel"/>
+  <origin xyz="0.25 0 -0.055" rpy="0 0 0"/> <!-- Adjust xyz as per the desired position -->
+</joint>
   <!-- Transmission for wheels -->
   <transmission name="left_wheel_trans">
@@ -154,11 +181,11 @@
           <samples>720</samples>
           <resolution>1</resolution>
-          <min_angle>0</min_angle>
-          <max_angle>1.570796</max_angle>
+          <min_angle>-3.14</min_angle>
+          <max_angle>3.14</max_angle>
         </horizontal>
       </scan>
       <range>
         <min>0.1</min>
-        <max>30.0</max>
+        <max>12</max>
         <resolution>0.01</resolution>
       </range>

Commit message: 2D Lidar to 3D Map

File: src/ugv_sim/urdf/ugv.urdf.xacro (robot description, xacro)
@@ -92,41 +92,58 @@
   </inertial>
 </link>
+  <link name="lidar_link">
+    <visual>
+      <geometry>
+        <box size="0.1 0.1 0.05"/> <!-- Size to be adjusted -->
+      </geometry>
+    </visual>
+    <inertial>
+      <mass value="1.0"/> <!-- Adjust mass -->
+      <inertia ixx="0.001" ixy="0" ixz="0" iyy="0.001" iyz="0" izz="0.001"/> <!-- Adjust inertia -->
+    </inertial>
+  </link>
+  <!-- Joints -->
+  <!-- Left Wheel Joint -->
+  <joint name="left_wheel_joint" type="continuous">
+    <parent link="base_link"/>
+    <child link="left_wheel"/>
+    <origin xyz="0.0 0.3 -0.02" rpy="1.5707 0 0"/>
+    <axis xyz="0 0 1"/>
+  </joint>
+  <!-- Right Wheel Joint -->
+  <joint name="right_wheel_joint" type="continuous">
+    <parent link="base_link"/>
+    <child link="right_wheel"/>
+    <origin xyz="0 -0.3 -0.02" rpy="1.5707 0 0"/>
+    <axis xyz="0 0 1"/>
+  </joint>
+  <!-- Front Joint -->
+  <joint name="front_wheel_joint" type="fixed">
+    <parent link="base_link"/>
+    <child link="front_wheel"/>
+    <origin xyz="0.25 0 -0.055" rpy="0 0 0"/> <!-- Adjust xyz as per the desired position -->
+  </joint>
+  <!-- Servo Motor Joint -->
+  <joint name="servo_joint" type="revolute">
+    <parent link="base_link"/>
+    <child link="lidar_link"/>
+    <origin xyz="0 0 0.1" rpy="0 0 0"/> <!-- Position to be adjusted -->
+    <axis xyz="0 1 0"/>
+    <limit lower="-1.57" upper="1.57" effort="5" velocity="1"/>
+  </joint>
+  <!-- Lidar Joint
+  <joint name="lidar_joint" type="fixed">
+    <parent link="base_link"/>
+    <child link="lidar_link"/>
+    <origin xyz="0 0 0.1" rpy="0 0 0"/>
+  </joint> -->
 <!-- Lidar Link -->
-<link name="lidar_link">
+<!-- <link name="lidar_link">
   <visual>
     <geometry>
       <cylinder length="0.1" radius="${wheel_radius}"/>
     </geometry>
-    <!-- Add material properties if desired -->
   </visual>
-</link>
-  <!-- Joints -->
-  <!-- Left Wheel Joint -->
-  <joint name="left_wheel_joint" type="continuous">
-    <parent link="base_link"/>
-    <child link="left_wheel"/>
-    <origin xyz="0.0 0.3 -0.02" rpy="1.5707 0 0"/>
-    <axis xyz="0 0 1"/>
-  </joint>
-  <!-- Right Wheel Joint -->
-  <joint name="right_wheel_joint" type="continuous">
-    <parent link="base_link"/>
-    <child link="right_wheel"/>
-    <origin xyz="0 -0.3 -0.02" rpy="1.5707 0 0"/>
-    <axis xyz="0 0 1"/>
-  </joint>
-  <!-- Lidar Joint -->
-  <joint name="lidar_joint" type="fixed">
-    <parent link="base_link"/>
-    <child link="lidar_link"/>
-    <!-- Define the origin of the joint -->
-    <origin xyz="0 0 0.1" rpy="0 0 0"/>
-  </joint>
-<!-- Front Joint -->
-<joint name="front_wheel_joint" type="fixed">
-  <parent link="base_link"/>
-  <child link="front_wheel"/>
-  <origin xyz="0.25 0 -0.055" rpy="0 0 0"/> <!-- Adjust xyz as per the desired position -->
-</joint>
+</link> -->
   <!-- Transmission for wheels -->
   <transmission name="left_wheel_trans">
@@ -150,4 +167,15 @@
     </actuator>
   </transmission>
+  <!-- Transmission for Servo Motor -->
+<transmission name="servo_transmission">
+  <type>transmission_interface/SimpleTransmission</type>
+  <joint name="servo_joint">
+    <hardwareInterface>PositionJointInterface</hardwareInterface>
+  </joint>
+  <actuator name="servo_motor">
+    <hardwareInterface>PositionJointInterface</hardwareInterface>
+    <mechanicalReduction>1</mechanicalReduction>
+  </actuator>
+</transmission>
 <gazebo>
     <plugin name="gazebo_ros_control" filename="libgazebo_ros_control.so">
@@ -156,5 +184,5 @@
       <legacyModeNS>true</legacyModeNS> -->
       <robotParam>robot_description</robotParam>
-      <controller name=" left_wheel_controller right_wheel_controller"/>
+      <controller name=" left_wheel_controller right_wheel_controller servo_controller"/>
     </plugin>
     <plugin name="p3d_base_controller" filename="libgazebo_ros_p3d.so">

Commit message: stuff

File: src/ugv_sim/urdf/ugv.urdf.xacro (robot description, xacro)
@@ -129,5 +129,5 @@
     <child link="lidar_link"/>
     <origin xyz="0 0 0.1" rpy="0 0 0"/> <!-- Position to be adjusted -->
-    <axis xyz="0 1 0"/>
+    <axis xyz="1 0 0"/>
     <limit lower="-1.57" upper="1.57" effort="5" velocity="1"/>
   </joint>

Commit message: Lidar Package Is Added

File: src/ugv_sim/urdf/ugv.urdf.xacro (robot description, xacro)
@@ -6,4 +6,10 @@
   <xacro:property name="chassis_radius" value="0.3"/>
   <xacro:property name="chassis_height" value="0.1"/>
+  <link name="base_footprint">
+  <inertial>
+    <mass value="0.0"/>
+    <inertia ixx="0.0" ixy="0.0" ixz="0.0" iyy="0.0" iyz="0.0" izz="0.0"/>
+  </inertial>
+</link>
   <!-- Base Link -->
   <link name="base_link">
@@ -104,4 +110,9 @@
   </link>
   <!-- Joints -->
+  <joint name="base_footprint_joint" type="fixed">
+  <parent link="base_link"/>
+  <child link="base_footprint"/>
+  <origin xyz="0 -0.2 0" rpy="0 0 0"/> <!-- Adjust the origin if necessary -->
+</joint>
   <!-- Left Wheel Joint -->
   <joint name="left_wheel_joint" type="continuous">
@@ -122,5 +133,5 @@
     <parent link="base_link"/>
     <child link="front_wheel"/>
-    <origin xyz="0.25 0 -0.055" rpy="0 0 0"/> <!-- Adjust xyz as per the desired position -->
+    <origin xyz="-0.25 0 -0.055" rpy="0 0 0"/> <!-- Adjust xyz as per the desired position -->
   </joint>
   <!-- Servo Motor Joint -->
@@ -184,5 +195,5 @@
       <legacyModeNS>true</legacyModeNS> -->
       <robotParam>robot_description</robotParam>
-      <controller name=" left_wheel_controller right_wheel_controller servo_controller"/>
+      <controller name=" diff_drive_controller servo_controller"/>
     </plugin>
     <plugin name="p3d_base_controller" filename="libgazebo_ros_p3d.so">
@@ -190,5 +201,5 @@
       <updateRate>50.0</updateRate>
       <bodyName>base_link</bodyName>
-      <topicName>odom</topicName>
+      <topicName>world</topicName>
       <publishOdomTF>true</publishOdomTF>
       <publishTf>true</publishTf>
